File: kicad/mini_scope/mini_scope.sch (KiCad schematic (older format))
At the start: 7 parts

Commit message: schematic complete
Parts:
- removed R?: R, symbol Device:R
- added C? (x2): 1u, symbol Device:C
- added C?: 1n, symbol Device:C
- added C? (x3): 10u, symbol Device:C
- added C? (x10): 100n, symbol Device:C
- added C? (x2): CP, symbol Device:CP
- added D?: 1N4007, Diode_THT:D_DO-41_SOD81_P10.16mm_Horizontal, symbol Diode:1N4007
- added D? (x2): LED, symbol Device:LED
- added J?: Conn_Coaxial, symbol Connector:Conn_Coaxial
- added J?: STK3700_exp_conn, symbol conn:STK3700_exp_conn
- added J?: USB_B_Mini, symbol Connector:USB_B_Mini
- added K?: EC2-5NU, Relay_THT:Relay_DPDT_Kemet_EC2, symbol Relay:EC2-5NU
- added Q?: BC848, Package_TO_SOT_SMD:SOT-23, symbol Transistor_BJT:BC848
- added R? (x2): 10k, symbol Device:R
- added R?: 1k, symbol Device:R
- added R?: 91k, symbol Device:R
- added R? (x2): 22, symbol Device:R
- added R? (x4): 470, symbol Device:R
- added R? (x2): 270, symbol Device:R
- added U?: ISL28134, symbol lib1:ISL28134
- added U?: FT232RL, Package_SO:SSOP-28_5.3x10.2mm_P0.65mm, symbol Interface_USB:FT232RL
- added U?: CRE1S0505SC, Converter_DCDC:Converter_DCDC_muRata_CRE1xxxxxxSC_THT, symbol Regulator_Switching:CRE1S0505SC
- added U? (x2): TLP2761, Package_SO:SO-6L_10x3.84mm_P1.27mm, symbol Isolator:TLP2761
- R?: value R -> 1k
- R?: value R -> 47k
- R?: value R -> 1M
Connections:
- net at U?.2 (-): now also R?.1, U?.6 (Vout)
- net at R?.1, U?.3 (+): now also D?.1 (K), D?.2 (A)
- net GND: now reaches D?.2 (A), U?.4 (V-)
- net GND: now also C?.2, C?.2, C?.2, C?.2, C?.2, C?.2, C?.2, C?.2, C?.2, J?.1 (GND), J?.19 (GND), Q?.2 (E), R?.2, R?.2, U?.3 (-VOUT), U?.4 (GND), U?.4 (V-); no longer R?.2
- net +5V: now reaches D?.1 (K), U?.7 (V+)
- net +5V: now also C?.1, C?.1, C?.1, C?.1, C?.1, C?.1, C?.1, C?.1, C?.1, D?.1 (K), J?.18 (5V), K?.1, R?.1, U?.4 (+VOUT), U?.7 (V+)
- net at R?.2: now also R?.1, C?.1, K?.8
- net GNDREF: now reaches R?.2
- net GNDREF: now also C?.2, C?.2, C?.2, J?.2 (Ext), U?.2 (-), U?.6 (Vout)
- new net: R?.1, R?.2, U?.3 (+)
- new net: C?.2, J?.1 (In), K?.9
- new net: Q?.1 (B), R?.1
- new net: D?.2 (A), K?.12, Q?.3 (C)
- new net: R?.2, U?.1 (TXD)
- new net: R?.2, U?.15 (USBD+)
- new net: R?.2, U?.16 (USBD-)
- new net: C?.1, U?.17 (3V3OUT)
- new net: D?.1 (K), U?.22 (CBUS1)
- new net: D?.1 (K), U?.23 (CBUS0)
- new net: R?.2, U?.5 (RXD)
- new net: J?.3 (D+), R?.1
- new net: J?.2 (D-), R?.1
- new net: R?.1, U?.5 (VO)
- new net: R?.1, U?.3 (K)
- new net: R?.2, U?.1 (A) (x2)
- new net: D?.2 (A), R?.1 (x2)
- new net +3V3: C?.1, C?.1, J?.20 (3V3), R?.1, U?.6 (VDD)
- new net Earth: C?.2, C?.2, C?.2, J?.5 (GND), J?.6 (Shield), U?.1 (-VIN), U?.18 (GND), U?.21 (GND), U?.25 (AGND), U?.26 (TEST), U?.4 (GND), U?.7 (GND)
- new net RX: U?.5 (VO)
- new net TO_ADC: C?.1, J?.10 (PD3), R?.1, R?.2
- new net TX: U?.3 (K)
- new net VBUS: C?.1, C?.1, J?.1 (VBUS), R?.1, R?.2, R?.2, U?.19 (~RESET~), U?.2 (+VIN), U?.20 (VCC), U?.4 (VCCIO), U?.6 (VDD)
- new net ac_dc_couple: J?.12 (PD4), R?.2
Other:
- note added: "ANALOG INPUT STAGE\n"
- note added: "FILTER CAPACITORS\n"
- note added: "POWER ISOLATION\n"
- note added: "POWER SUPPLY SPLIT\n"
- note added: "SERIAL ISOLATION"
- note added: "STK3700 CONNECTOR\n"
- note added: "USB-TO-SERIAL"
- moved on the sheet: D?, R?, U?

Commit message: almost finished pcb
Parts:
- removed C?: CP, symbol Device:CP
- removed D?: LED, symbol Device:LED
- removed J?: USB_B_Mini, symbol Connector:USB_B_Mini
- removed K?: EC2-5NU, Relay_THT:Relay_DPDT_Kemet_EC2, symbol Relay:EC2-5NU
- removed R? (x2): 22, symbol Device:R
- removed R?: 470, symbol Device:R
- removed U? (x2): ISL28134, symbol lib1:ISL28134
- added C1, C2: 100n, Capacitor_SMD:C_0805_2012Metric_Pad1.18x1.45mm_HandSolder, symbol Device:C
- added C12: 470u, Capacitor_SMD:CP_Elec_8x10.5, symbol Device:CP
- added D4, D6, D7, D9: LED, LED_SMD:LED_0805_2012Metric_Pad1.15x1.40mm_HandSolder, symbol Device:LED
- added F1, F2: Polyfuse_Small, Resistor_SMD:R_1206_3216Metric_Pad1.30x1.75mm_HandSolder, symbol Device:Polyfuse_Small
- added FB?: Ferrite_Bead_Small, Resistor_SMD:R_0805_2012Metric_Pad1.20x1.40mm_HandSolder, symbol Device:Ferrite_Bead_Small
- added H1, H2, H3, H4: MountingHole, MountingHole:MountingHole_3.2mm_M3_DIN965_Pad, symbol Mechanical:MountingHole
- added J1: USB_B_Mini, mini_scope:usb_b_mini, symbol lib1:USB_B_Mini
- added J3, J?: Conn_01x03_Male, Connector_PinHeader_2.54mm:PinHeader_1x03_P2.54mm_Vertical, symbol Connector:Conn_01x03_Male
- added K1: G5LE-1, mini_scope:Relay_SPDT_Omron-G5LE-1, symbol Relay:G5LE-1
- added R17: 470, Resistor_SMD:R_0805_2012Metric_Pad1.20x1.40mm_HandSolder, symbol Device:R
- added R18, R19, R21: 270, Resistor_SMD:R_0805_2012Metric_Pad1.20x1.40mm_HandSolder, symbol Device:R
- added R5: 1k, Resistor_SMD:R_0805_2012Metric_Pad1.20x1.40mm_HandSolder, symbol Device:R
- added U2, U3: OPA340UA, Package_SO:SOIC-8_3.9x4.9mm_P1.27mm, symbol Amplifier_Operational:OPA340UA
- C10, C11, C18: renamed from C?; footprint (none) -> Capacitor_SMD:C_1210_3225Metric_Pad1.33x2.70mm_HandSolder
- C13, C14, C15, C17, C19, C20, C3, C4, C5, C6, C7, C9: renamed from C?; footprint (none) -> Capacitor_SMD:C_0805_2012Metric_Pad1.18x1.45mm_HandSolder
- C16: renamed from C?; value CP -> 470u; footprint (none) -> Capacitor_SMD:CP_Elec_8x10.5
- C8: renamed from C?; value 1u -> 10u; footprint (none) -> Capacitor_SMD:C_1210_3225Metric_Pad1.33x2.70mm_HandSolder
- D2, D3: renamed from D?; footprint (none) -> Diode_SMD:D_MicroMELF_Handsoldering
- D5: renamed from D?; footprint (none) -> LED_SMD:LED_0805_2012Metric_Pad1.15x1.40mm_HandSolder
- J2: renamed from J?; footprint (none) -> mini_scope:BNC_Amphenol_B6252HB-NPP3G-50_Horizontal
- J4: renamed from J?; footprint (none) -> Connector_PinSocket_2.54mm:PinSocket_2x10_P2.54mm_Horizontal
- R10, R11, R12, R16, R6, R8, R9: renamed from R?; footprint (none) -> Resistor_SMD:R_0805_2012Metric_Pad1.20x1.40mm_HandSolder
- R14: renamed from R?; value 47k -> 1k 1%; footprint (none) -> Resistor_SMD:R_0805_2012Metric_Pad1.20x1.40mm_HandSolder
- R15: renamed from R?; value 91k -> 1k 1%; footprint (none) -> Resistor_SMD:R_0805_2012Metric_Pad1.20x1.40mm_HandSolder
- R3, R4: renamed from R?; value 10k -> 1k 1%; footprint (none) -> Resistor_SMD:R_0805_2012Metric_Pad1.20x1.40mm_HandSolder
- R7: renamed from R?; value 1M -> 1M 1%; footprint (none) -> Resistor_SMD:R_0805_2012Metric_Pad1.20x1.40mm_HandSolder
- gave numbers to parts that had none: 6
Connections:
- net +3V3: now also R19.2
- net +5V: now also C16.1, C1.1, K1.5, R21.2, U2.7 (V+), U3.7 (V+)
- net Earth: now also C3.1, C12.2, J1.5 (GND), J1.6 (Shield), J1.7 (Shield); no longer C3.2
- net GND: now also C16.2, C2.2, D6.1 (K), D9.1 (K), J?.3 (Pin_3), U2.4 (V-), U3.4 (V-); no longer C5.2
- net GNDREF: now also C5.2, J3.3 (Pin_3), J?.1 (Pin_1)
- net RX: now also J4.6 (PD1), R17.2; no longer U4.5 (VO)
- net TO_ADC: no longer C5.1
- net TX: now also J4.4 (PD0)
- net VBUS: now also U4.1 (A), C12.1, FB?.1
- net at R14.1: now also U3.2 (-), U3.6
- net at D2.2 (A), D3.1 (K): now also F2.1, U3.3 (+); no longer R8.1
- net at C4.1, R7.1, R8.2: now also K1.3
- net at R3.2, R4.1: now also C1.2, C2.1, U2.3 (+)
- net at J2.1 (In): now also J3.1 (Pin_1); no longer C4.2
- net at D1.2 (A), Q1.3 (C): now also R5.2
- net RUN: now reaches J4.9 (PC5)
- net RUN: now also D7.1 (K), R18.2
- net at U1.15 (USBD+): now also J1.3 (D+)
- net at U1.16 (USBD-): now also J1.2 (D-)
- net at U1.17 (3V3OUT): now also C3.2; no longer C3.1
- net at U1.22 (CBUS1): now also D4.1 (K)
- net at R9.1: now also D4.2 (A)
- new net: C5.1, F2.2, R8.1
- new net: C4.2, J3.2 (Pin_2), K1.1
- new net: F1.2, U2.2 (-), U2.6
- new net: F1.1, J?.2 (Pin_2)
- new net: R17.1, U4.5 (VO)
- new net: K1.2, R5.1
- new net: FB?.2, J1.1 (VBUS)
- new net: D9.2 (A), R21.1
- new net: D7.2 (A), R19.1
- new net: D6.2 (A), R18.1
Other:
- note added: "Status leds\n"
- note added: "TODO \nTVS\nUSB - 5V protection diode\nPCB-re tervezni a módosítást"
- moved on the sheet: C11, C16, C17, C18, C19, C20, C3, C5, C9, D2, D3, R14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

Commit message: project refresh
Parts:
- removed R5: 1k, Resistor_SMD:R_0805_2012Metric_Pad1.20x1.40mm_HandSolder, symbol Device:R
- removed U4, U5: TLP2761, Package_SO:SO-6L_10x3.84mm_P1.27mm, symbol Isolator:TLP2761
- added D8: D_Schottky, Diode_SMD:D_SMA, symbol Device:D_Schottky
- added FB2: Ferrite_Bead_Small, Resistor_SMD:R_0805_2012Metric_Pad1.20x1.40mm_HandSolder, symbol Device:Ferrite_Bead_Small
- added J6: Conn_01x02_Male, Connector_PinHeader_2.54mm:PinHeader_1x02_P2.54mm_Vertical, symbol Connector:Conn_01x02_Male
- added U4: USBLC6-2SC6, Package_TO_SOT_SMD:SOT-23-6, symbol lib1:USBLC6-2SC6
- added U5, U7: TLP2368, Package_SO:SO-5_4.4x3.6mm_P1.27mm, symbol lib1:TLP2368
- R14, R15, R3, R4: value 1k 1% -> 2k2 1%
- U1: footprint Package_SO:SSOP-28_5.3x10.2mm_P0.65mm -> mini_scope:SSOP-28_5.3x10.2mm_P0.65mm
- gave numbers to parts that had none: 2
Connections:
- net +3V3: now also U5.6 (VDD)
- net +5V: now also D8.1 (K), J6.1 (Pin_1); no longer U6.4 (+VOUT)
- net Earth: now also FB2.1, U4.2 (GND), U7.4 (GND); no longer J1.5 (GND), J1.6 (Shield), J1.7 (Shield)
- net GND: now also U5.4 (GND)
- net GNDREF: now also J5.2 (Pin_2); no longer J5.1 (Pin_1)
- net TX: now also U7.3 (K)
- net VBUS: now also FB1.2, U4.5 (VBUS), U5.1 (A), U7.6 (VDD); no longer FB1.1
- net at D1.2 (A), Q1.3 (C): now also K1.2
- net at U1.15 (USBD+): now also U4.1 (I/O1); no longer J1.3 (D+)
- net at U1.16 (USBD-): now also U4.3 (I/O2); no longer J1.2 (D-)
- net at F1.1: now also J5.1 (Pin_1); no longer J5.2 (Pin_2)
- net at R10.1: now also U7.5 (VO)
- net at R12.1: now also U5.3 (K)
- net at R17.1: now also U5.5 (VO)
- net at R16.2: now also U7.1 (A)
- net at J1.1 (VBUS): now also FB1.1; no longer FB1.2
- new net: D8.2 (A), J6.2 (Pin_2), U6.4 (+VOUT)
- new net: J1.2 (D-), U4.4 (I/O2)
- new net: J1.3 (D+), U4.6 (I/O1)
- new net: FB2.2, J1.5 (GND), J1.6 (Shield), J1.7 (Shield)
Other:
- note added: "STATUS LEDS\n"
- note removed: "Status leds\n"
- note removed: "TODO \nTVS\nUSB - 5V protection diode\nPCB-re tervezni a módosítást"
- moved on the sheet: C11, C12, C16, C18, C20, C3, C9, D4, D5, D6, D7, D9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
